File: ob-xa-2p-lpf.sch (EAGLE design)
At the start: 0 parts

Commit message: make schematic
Parts:
- added AUDIO_IN, AUDIO_OUT, FREQ_CV, RES_CV: OFFBOARD2JACKALT, aarons_library:OFFBOARD2JACKALT
- added C1, C3: 15u, rcl:CPOL-EUE1.8-4
- added C2, C4, C5: 300p, rcl:C-EU050-025X075
- added C6: 100p, rcl:C-EU050-025X075
- added D1, D2, D3: 1N4148, adafruit:DIODEDO-1N4148
- added IC1: AS3320, analog_audio:AS3320
- added R1, R11, R13, R14, R2, R3, R4, R5: 100k, rcl:R-US_0207/10
- added R10: 91k, rcl:R-US_0207/10
- added R12: 300k, rcl:R-US_0207/10
- added R15: 270, rcl:R-US_0207/10
- added R16: 18k, rcl:R-US_0207/10
- added R17: 75k, rcl:R-US_0207/10
- added R18, R7: 33k, rcl:R-US_0207/10
- added R19: 10k, pot:TRIM_US-B64Y
- added R20: 44.2k, rcl:R-US_0207/10
- added R21: 1k, rcl:R-US_0207/10
- added R6: 500k, pot:TRIM_US-B64Y
- added R8: 220k, rcl:R-US_0207/10
- added R9: 330k, rcl:R-US_0207/10
Connections:
- new net +15V: IC1.VCC, R18.1
- new net -5V: R15.1, R9.2
- new net 0V: AUDIO_IN.GND, AUDIO_OUT.GND, C2.1, C4.2, C5.2, D3.C, FREQ_CV.GND, IC1.GND, R1.1, R21.1, RES_CV.GND
- new net AUDIO_IN: AUDIO_IN.SIGNAL, C1.+
- new net AUDIO_OUT: AUDIO_OUT.SIGNAL, IC1.OUT3, R10.1
- new net CFI: IC1.VCFI, R20.1, R21.2
- new net FREQ_CV: FREQ_CV.SIGNAL, R19.S
- new net N$1: R2.1, R3.1
- new net N$10: IC1.IN3, R13.2
- new net N$11: IC1.OUT4, R14.2
- new net N$12: IC1.IN4, R14.1
- new net N$13: IC1.VRES, R8.2
- new net N$14: C3.-, R12.1, R17.1, R8.1
- new net N$15: R12.2, R6.S
- new net N$16: IC1.VEE, R15.2
- new net N$17: IC1.IRES, R7.1, R9.1
- new net N$18: C4.1, IC1.CAP4
- new net N$19: R7.2, RES_CV.SIGNAL
- new net N$2: R19.A, R20.2
- new net N$20: C5.1, IC1.CAP3
- new net N$3: IC1.IN2, R11.2, R3.2, R5.2
- new net N$4: C2.2, IC1.CAP2
- new net N$5: IC1.OUT1, R4.1, R5.1
- new net N$6: C3.+, IC1.OUT2, R13.1
- new net N$7: C6.1, D1.A, D2.C, R11.1
- new net N$8: C6.2, D1.C, D2.A, R16.2, R17.2
- new net N$9: D3.A, R16.1, R18.2
- new net VIN: C1.-, IC1.IN1, R1.2, R10.2, R2.2, R4.2, R6.A
