File: ob-xa-2p-lpf.brd (EAGLE design)
At the start: 50.8 x 85.5 mm, 53 parts, among them IC1 AS3320, IC3 TL082P

Commit message: bit more layout cleanup
Parts:
- moved R8 7.74 mm to (14.5, 36.8), turned to 90 degrees
- moved RES 4.82 mm to (6.86, 36.8), turned to 90 degrees
- moved C10 4.44 mm to (40.6, 51.8)
- moved R7 4.06 mm to (11.4, 36.8), turned to 270 degrees
- moved C11 3.10 mm to (40.6, 44.2)
- moved R17 3.06 mm to (14.5, 69.6)
- moved RES_ADJ 3.06 mm to (25.4, 74.9)
- moved C5 3.06 mm to (36.3, 51.8)
- moved C3 3.06 mm to (7.37, 49.3)
- moved R11 3.06 mm to (11.4, 61.5)
- moved R13 3.06 mm to (17.5, 41.4)
- moved R2 3.06 mm to (17.5, 61.5)
- moved R3 3.06 mm to (14.5, 61.5)
- moved R4 3.06 mm to (11.4, 49.3)
- moved R5 3.06 mm to (14.5, 49.3)
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
Commit message: route everything
Parts:
- moved RES 5.11 mm to (6.35, 31.8), turned to 0 degrees
- moved C1 0.80 mm to (45.0, 69.8)
- moved C3 0.51 mm to (6.86, 49.3), turned to 180 degrees
- moved C12 0.51 mm to (9.40, 20.8)
- renumbered POWER_IN to PWR_IN
Routing:
- net 0V: track 0.00 -> 211.1 mm
- net +15V: track 0.00 -> 122.8 mm
- net -15V: track 0.00 -> 66.5 mm
- net VIN: track 0.00 -> 47.2 mm
- net N$14: track 0.00 -> 45.6 mm
- net N$23: track 0.00 -> 38.3 mm
- net N$10: track 0.00 -> 29.1 mm
- net CFI: track 0.00 -> 28.0 mm
- net AUDIO_OUT: track 0.00 -> 21.7 mm
- net N$12: track 0.00 -> 19.2 mm
- net N$2: track 0.00 -> 17.3 mm
- net N$11: track 0.00 -> 17.1 mm
- net N$8: track 0.00 -> 15.3 mm
- net N$6: track 0.00 -> 15.2 mm
- net N$7: track 0.00 -> 14.8 mm
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
Commit message: add mounting holes
Parts:
- moved C1 4.32 mm to (45.0, 74.2)
- moved C11 4.32 mm to (40.6, 48.5)
- moved C2 4.32 mm to (17.5, 55.9)
- moved C4 4.32 mm to (36.3, 48.5)
- moved D3 4.32 mm to (25.7, 68.1)
- moved R7 4.32 mm to (11.4, 41.1)
- moved R8 4.32 mm to (14.5, 41.1)
- moved C12 4.32 mm to (9.40, 25.1)
- moved C13 4.32 mm to (4.32, 25.1)
- moved CV2 4.32 mm to (47.0, 25.9)
- moved FREQ_CV_2 4.32 mm to (47.5, 34.8)
- moved V/OCT_ADJ 4.32 mm to (25.4, 30.5)
- moved R25 4.32 mm to (37.1, 10.2)
- moved R6 4.32 mm to (25.4, 10.2)
- moved C14 4.32 mm to (18.0, 14.5)
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Other:
- board size 50.8 x 85.5 mm -> 50.8 x 88.9 mm
- board text added: "+15 GND -15"
- board text added: ">LAST_DATE_TIME"
- board text added: "OB-XA-2P-LFP Board: Ben Terry ACMS Spring 2020"
- board text added: "Square pads of panel jumpers are Ground"

Commit message: minor cleanup. Draft2 rev
Routing:
- net -15V: track 66.5 -> 67.2 mm
